File: DriverBoard/DriverBoard.sch (KiCad schematic (older format))
At the start: 27 parts, among them U1 TPS92510, U2 RT9058-50GV, U3 74AHCT1G125

Commit message: pcb: r0p1
Parts:
- DIM1, ENA1, GND1, LED+1, LED-1, VCC1: footprint TestPoint:TestPoint_Pad_3.0x3.0mm -> TestPoint:TestPoint_Pad_1.5x1.5mm
- L1: footprint Inductor_SMD:L_Bourns_SRP7028A_7.3x6.6mm -> Footprints:L_7.1x6.6mm
Connections:
- net at C6.2, R5.2, U1.7 (VSENSE): now also RB1.3; no longer RB1.1
- net at RA1.1: now also R3.1, RA1.2; no longer RB1.3
- new net: RA1.3, RB1.1
Changed lines of the file:
@@
 F 0 "VCC1" H 4200 3300 50  0000 C CNN
 F 1 "Conn_01x01" H 3918 3166 50  0001 C CNN
-F 2 "TestPoint:TestPoint_Pad_3.0x3.0mm" H 4000 3300 50  0001 C CNN
+F 2 "TestPoint:TestPoint_Pad_1.5x1.5mm" H 4000 3300 50  0001 C CNN
 F 3 "~" H 4000 3300 50  0001 C CNN
 	1    4000 3300
@@
 F 0 "ENA1" H 4200 3800 50  0000 C CNN
 F 1 "Conn_01x01" H 3918 3666 50  0001 C CNN
-F 2 "TestPoint:TestPoint_Pad_3.0x3.0mm" H 4000 3800 50  0001 C CNN
+F 2 "TestPoint:TestPoint_Pad_1.5x1.5mm" H 4000 3800 50  0001 C CNN
 F 3 "~" H 4000 3800 50  0001 C CNN
 	1    4000 3800
@@
 F 0 "DIM1" H 4200 4300 50  0000 C CNN
 F 1 "Conn_01x01" H 3918 4166 50  0001 C CNN
-F 2 "TestPoint:TestPoint_Pad_3.0x3.0mm" H 4000 4300 50  0001 C CNN
+F 2 "TestPoint:TestPoint_Pad_1.5x1.5mm" H 4000 4300 50  0001 C CNN
 F 3 "~" H 4000 4300 50  0001 C CNN
 	1    4000 4300
@@
 F 0 "GND1" H 4200 4800 50  0000 C CNN
 F 1 "Conn_01x01" H 3918 4666 50  0001 C CNN
-F 2 "TestPoint:TestPoint_Pad_3.0x3.0mm" H 4000 4800 50  0001 C CNN
+F 2 "TestPoint:TestPoint_Pad_1.5x1.5mm" H 4000 4800 50  0001 C CNN
 F 3 "~" H 4000 4800 50  0001 C CNN
 	1    4000 4800
@@
 F 0 "L1" V 7475 3300 50  0000 C CNN
 F 1 "33uH" V 7384 3300 50  0000 C CNN
-F 2 "Inductor_SMD:L_Bourns_SRP7028A_7.3x6.6mm" H 7250 3300 50  0001 C CNN
+F 2 "Footprints:L_7.1x6.6mm" H 7250 3300 50  0001 C CNN
 F 3 "~" H 7250 3300 50  0001 C CNN
 	1    7250 3300
@@
 F 0 "LED+1" H 8000 3300 50  0000 C CNN
 F 1 "Conn_01x01" H 7718 3166 50  0001 C CNN
-F 2 "TestPoint:TestPoint_Pad_3.0x3.0mm" H 7800 3300 50  0001 C CNN
+F 2 "TestPoint:TestPoint_Pad_1.5x1.5mm" H 7800 3300 50  0001 C CNN
 F 3 "~" H 7800 3300 50  0001 C CNN
 	1    7800 3300
@@
 F 0 "LED-1" H 8000 4800 50  0000 C CNN
 F 1 "Conn_01x01" H 7718 4666 50  0001 C CNN
-F 2 "TestPoint:TestPoint_Pad_3.0x3.0mm" H 7800 4800 50  0001 C CNN
+F 2 "TestPoint:TestPoint_Pad_1.5x1.5mm" H 7800 4800 50  0001 C CNN
 F 3 "~" H 7800 4800 50  0001 C CNN
 	1    7800 4800
@@
 F 3 "~" H 6250 4350 50  0001 C CNN
 	1    6250 4350
-	0    1    1    0
+	0    -1   1    0
 $EndComp
 Wire Wire Line
@@
 F 3 "~" H 6550 4350 50  0001 C CNN
 	1    6550 4350
-	0    1    1    0
-$EndComp
-Wire Wire Line
+	0    -1   1    0
+$EndComp
+Wire Wire Line
